Commit message: robotic_manip_3 now working, rviz config updated

File: robotic_manip_3/urdf/robotic_manip_3.urdf (robot description, URDF)
Before this commit: robot robotic_manip_3, 5 links, 4 joints
Links:
- link base_link: geometry visual cylinder length=0.1 radius=0.1
- link link_1: geometry visual box size=0.01 0.01 0.4
- link link_2: geometry visual box size=0.01 0.01 0.2
- link link_3: geometry visual box size=0.01 0.01 0.2
Joints:
- joint joint_1: origin xyz=0 0 10 rpy=0 0 0 -> xyz=0 0 0.1 rpy=0 0 0
- joint joint_2: origin xyz=0 0 40 rpy=0 0 0 -> xyz=0 0 0.4 rpy=0 0 0
- joint joint_3: origin xyz=0 0 10 rpy=0 0 0 -> xyz=0 0 0.2 rpy=0 0 0
- joint joint_ee: origin xyz=0 0 20 rpy=0 0 0 -> xyz=0 0 0.2 rpy=0 0 0
