Commit message: 6DOF robot?

File: serial_link_robot/urdf/serial_link_robot.urdf (robot description, URDF)
Before this commit: robot serial_link_robot, 5 links, 4 joints
Links:
- added link link_4; collision cylinder length=0.11 radius=0.04; visual cylinder length=0.11 radius=0.04
- added link link_5; collision cylinder length=0.095 radius=0.035; visual cylinder length=0.095 radius=0.035
- added link link_6; collision cylinder length=0.083 radius=0.03; visual cylinder length=0.083 radius=0.03
- link base_link: geometry collision cylinder length=0.09 radius=0.09; visual cylinder length=0.09 radius=0.09
- link link_1: geometry collision cylinder length=0.16 radius=0.075; visual cylinder length=0.16 radius=0.075
- link link_2: geometry collision cylinder length=0.425 radius=0.055; visual cylinder length=0.425 radius=0.055
- link link_3: geometry collision cylinder length=0.392 radius=0.05; visual cylinder length=0.392 radius=0.05
- link link_ee: geometry collision cylinder length=0.06 radius=0.028; visual cylinder length=0.06 radius=0.028
Joints:
- added joint joint_4: type revolute, parent link_3, child link_4, origin xyz=0 0 0.392 rpy=0 0 0, axis 1 0 0, limit lower=-6.283 upper=6.283 effort=80 velocity=2.0
- added joint joint_5: type revolute, parent link_4, child link_5, origin xyz=0 0 0.11 rpy=0 0 0, axis 0 1 0, limit lower=-6.283 upper=6.283 effort=60 velocity=2.5
- added joint joint_6: type revolute, parent link_5, child link_6, origin xyz=0 0 0.095 rpy=0 0 0, axis 0 0 1, limit lower=-6.283 upper=6.283 effort=40 velocity=3.0
- joint joint_1: limit lower=-3.14 upper=3.14 effort=100.0 velocity=0.5 -> lower=-6.283 upper=6.283 effort=150 velocity=1.5; origin xyz=0 0 0.2 rpy=0 0 0 -> xyz=0 0 0.09 rpy=0 0 0
- joint joint_2: axis 1 0 0 -> 0 1 0; limit lower=-3.14 upper=3.14 effort=100.0 velocity=0.5 -> lower=-3.14 upper=3.14 effort=150 velocity=1.5; origin xyz=0 0 0.4 rpy=0 0 0 -> xyz=0 0 0.16 rpy=0 0 0
- joint joint_3: axis 1 0 0 -> 0 1 0; limit lower=-3.14 upper=3.14 effort=100.0 velocity=0.5 -> lower=-3.14 upper=3.14 effort=120 velocity=1.5; origin xyz=0 0 0.5 rpy=0 0 0 -> xyz=0 0 0.425 rpy=0 0 0
- joint joint_ee: origin xyz=0 0.6 0 rpy=0 0 0 -> xyz=0 0 0.083 rpy=0 0 0; parent link_3 -> link_6
